File: Board/RevA/IMU.sch (KiCad schematic (older format))
At the start: 1 part

Commit message: Finished Rough RevA and Added Annotations
Parts:
- gave numbers to parts that had none: 1
Changed lines of the file:
@@
 $EndDescr
 $Comp
-L Connector:Conn_01x06_Male J?
+L Connector:Conn_01x06_Male J1
 U 1 1 614AF895
 P 4300 3500
-F 0 "J?" H 4408 3881 50  0000 C CNN
+AR Path="/614ADF24/614AF895" Ref="J1"  Part="1"
+AR Path="/614AE184/614AF895" Ref="J2"  Part="1"
+F 0 "J2" H 4408 3881 50  0000 C CNN
 F 1 "Conn_01x06_Male" H 4408 3790 50  0000 C CNN
 F 2 "" H 4300 3500 50  0001 C CNN

Commit message: Added Footprints to RevA 1/2
Changed lines of the file:
@@
 $Descr A4 11693 8268
 encoding utf-8
-Sheet 3 5
+Sheet 2 5
 Title ""
 Date ""
@@
 AR Path="/614ADF24/614AF895" Ref="J1"  Part="1"
 AR Path="/614AE184/614AF895" Ref="J2"  Part="1"
-F 0 "J2" H 4408 3881 50  0000 C CNN
+F 0 "J1" H 4408 3881 50  0000 C CNN
 F 1 "Conn_01x06_Male" H 4408 3790 50  0000 C CNN
 F 2 "" H 4300 3500 50  0001 C CNN

Commit message: Updated Power Pins and Header Layout
Parts:
- J1: footprint (none) -> Connector_PinHeader_2.54mm:PinHeader_1x06_P2.54mm_Horizontal
Changed lines of the file:
@@
 $Descr A4 11693 8268
 encoding utf-8
-Sheet 2 5
+Sheet 3 5
 Title ""
 Date ""
@@
 AR Path="/614ADF24/614AF895" Ref="J1"  Part="1"
 AR Path="/614AE184/614AF895" Ref="J2"  Part="1"
-F 0 "J1" H 4408 3881 50  0000 C CNN
+F 0 "J2" H 4408 3881 50  0000 C CNN
 F 1 "Conn_01x06_Male" H 4408 3790 50  0000 C CNN
-F 2 "" H 4300 3500 50  0001 C CNN
+F 2 "Connector_PinHeader_2.54mm:PinHeader_1x06_P2.54mm_Horizontal" H 4300 3500 50  0001 C CNN
 F 3 "~" H 4300 3500 50  0001 C CNN
 	1    4300 3500
