File: Board/RevA/p21014.sch (KiCad schematic (older format))
At the start: 10 parts, among them SW1 SW_Push

Commit message: Added Footprints to RevA 1/2
Parts:
- BT1: footprint (none) -> 0_MSD_FPs:AJS-Coin-Cell_1062-Digikey
- D1: footprint (none) -> 0_MSD_FPs:RGB_AJS
- D2: footprint (none) -> LED_SMD:LED_1812_4532Metric
- R1, R2, R3, R4, R5, R6: footprint (none) -> Resistor_SMD:R_0603_1608Metric
Changed lines of the file:
@@
 F 0 "BT1" H 3918 1946 50  0000 L CNN
 F 1 "Battery_Cell" H 3918 1855 50  0000 L CNN
-F 2 "" V 3800 1910 50  0001 C CNN
+F 2 "0_MSD_FPs:AJS-Coin-Cell_1062-Digikey" V 3800 1910 50  0001 C CNN
 F 3 "~" V 3800 1910 50  0001 C CNN
 	1    3800 1850
@@
 F 0 "D2" V 5189 2032 50  0000 R CNN
 F 1 "LED" V 5098 2032 50  0000 R CNN
-F 2 "" H 5150 2150 50  0001 C CNN
+F 2 "LED_SMD:LED_1812_4532Metric" H 5150 2150 50  0001 C CNN
 F 3 "~" H 5150 2150 50  0001 C CNN
 	1    5150 2150
@@
 F 0 "R4" H 5218 1796 50  0000 L CNN
 F 1 "350" H 5218 1705 50  0000 L CNN
-F 2 "" V 5190 1740 50  0001 C CNN
+F 2 "Resistor_SMD:R_0603_1608Metric" V 5190 1740 50  0001 C CNN
 F 3 "~" H 5150 1750 50  0001 C CNN
 	1    5150 1750
@@
 F 0 "R5" H 6518 3796 50  0000 L CNN
 F 1 "10k" H 6518 3705 50  0000 L CNN
-F 2 "" V 6490 3740 50  0001 C CNN
+F 2 "Resistor_SMD:R_0603_1608Metric" V 6490 3740 50  0001 C CNN
 F 3 "~" H 6450 3750 50  0001 C CNN
 	1    6450 3750
@@
 F 0 "R6" H 6518 4096 50  0000 L CNN
 F 1 "10k" H 6518 4005 50  0000 L CNN
-F 2 "" V 6490 4040 50  0001 C CNN
+F 2 "Resistor_SMD:R_0603_1608Metric" V 6490 4040 50  0001 C CNN
 F 3 "~" H 6450 4050 50  0001 C CNN
 	1    6450 4050
@@
 F 0 "D1" H 4650 6647 50  0000 C CNN
 F 1 "LED_RGB" H 4650 6556 50  0000 C CNN
-F 2 "" H 4650 6100 50  0001 C CNN
+F 2 "0_MSD_FPs:RGB_AJS" H 4650 6100 50  0001 C CNN
 F 3 "~" H 4650 6100 50  0001 C CNN
 	1    4650 6150
@@
 F 0 "R2" H 4368 5996 50  0000 L CNN
 F 1 "350" H 4368 5905 50  0000 L CNN
-F 2 "" V 4340 5940 50  0001 C CNN
+F 2 "Resistor_SMD:R_0603_1608Metric" V 4340 5940 50  0001 C CNN
 F 3 "~" H 4300 5950 50  0001 C CNN
 	1    4300 5950
@@
 F 0 "R1" H 4018 6196 50  0000 L CNN
 F 1 "350" H 4018 6105 50  0000 L CNN
-F 2 "" V 3990 6140 50  0001 C CNN
+F 2 "Resistor_SMD:R_0603_1608Metric" V 3990 6140 50  0001 C CNN
 F 3 "~" H 3950 6150 50  0001 C CNN
 	1    3950 6150
@@
 F 0 "R3" H 4368 6396 50  0000 L CNN
 F 1 "350" H 4368 6305 50  0000 L CNN
-F 2 "" V 4340 6340 50  0001 C CNN
+F 2 "Resistor_SMD:R_0603_1608Metric" V 4340 6340 50  0001 C CNN
 F 3 "~" H 4300 6350 50  0001 C CNN
 	1    4300 6350

Commit message: Updated Power Pins and Header Layout
Parts:
- SW1: footprint (none) -> 0_MSD_FPs:AJS-Switch_CFS-0102TA
Changed lines of the file:
@@
 F 0 "SW1" H 4200 1735 50  0000 C CNN
 F 1 "SW_Push" H 4200 1644 50  0000 C CNN
-F 2 "" H 4200 1650 50  0001 C CNN
+F 2 "0_MSD_FPs:AJS-Switch_CFS-0102TA" H 4200 1650 50  0001 C CNN
 F 3 "~" H 4200 1650 50  0001 C CNN
 	1    4200 1450
