File: Board/RevB/IMU.sch (KiCad schematic (older format))
At the start: 1 part, among them J1 Conn_01x06_Male

Commit message: Updated RevB Schematic
Parts:
- J1: footprint Connector_PinHeader_2.54mm:PinHeader_1x06_P2.54mm_Horizontal -> 0_MSD_FPs:MSD_6_Pin
Connections:
- net SCL: now also J1.5 (Pin_5); no longer J1.4 (Pin_4)
- net SDA: now also J1.4 (Pin_4); no longer J1.5 (Pin_5)
Changed lines of the file:
@@
 $Descr A4 11693 8268
 encoding utf-8
-Sheet 3 5
+Sheet 2 4
 Title ""
 Date ""
@@
 AR Path="/614ADF24/614AF895" Ref="J1"  Part="1"
 AR Path="/614AE184/614AF895" Ref="J2"  Part="1"
-F 0 "J2" H 4408 3881 50  0000 C CNN
+F 0 "J1" H 4408 3881 50  0000 C CNN
 F 1 "Conn_01x06_Male" H 4408 3790 50  0000 C CNN
-F 2 "Connector_PinHeader_2.54mm:PinHeader_1x06_P2.54mm_Horizontal" H 4300 3500 50  0001 C CNN
+F 2 "0_MSD_FPs:MSD_6_Pin" H 4300 3500 50  0001 C CNN
 F 3 "~" H 4300 3500 50  0001 C CNN
 	1    4300 3500
@@
 Text HLabel 4500 3500 2    50   Input ~ 0
 GND
+Text HLabel 4500 3700 2    50   BiDi ~ 0
+SCL
 Text HLabel 4500 3600 2    50   BiDi ~ 0
-SCL
-Text HLabel 4500 3700 2    50   BiDi ~ 0
 SDA
 Text HLabel 4500 3800 2    50   Input ~ 0
