File: Board/RevB/p21014.sch (KiCad schematic (older format))
At the start: 10 parts, among them SW1 SW_Push

Commit message: Updated RevB Schematic
Connections:
- no-connect marks 2 -> 1
Changed lines of the file:
@@
 $Descr A4 11693 8268
 encoding utf-8
-Sheet 1 5
+Sheet 1 4
 Title ""
 Date ""
@@
 F7 "RST" I R 9250 4250 50
 $EndSheet
-$Sheet
-S 8000 1450 1200 950
-U 614AE184
-F0 "IMU_B" 50
-F1 "IMU.sch" 50
-F2 "Vin" I L 8000 1700 50
-F3 "3v" O L 8000 1900 50
-F4 "GND" I L 8000 2150 50
-F5 "SCL" B R 9200 1700 50
-F6 "SDA" B R 9200 1900 50
-F7 "RST" I R 9200 2100 50
-$EndSheet
-$Comp
-L power:GNDREF #PWR0101
-U 1 1 614B1DB7
-P 7650 2300
-F 0 "#PWR0101" H 7650 2050 50  0001 C CNN
-F 1 "GNDREF" H 7655 2127 50  0000 C CNN
-F 2 "" H 7650 2300 50  0001 C CNN
-F 3 "" H 7650 2300 50  0001 C CNN
-	1    7650 2300
-	1    0    0    -1
-$EndComp
 $Comp
 L power:GNDREF #PWR0102
@@
 Wire Wire Line
 	7750 4300 7750 4450
-Wire Wire Line
-	7650 2150 8000 2150
-Wire Wire Line
-	7650 2150 7650 2300
 Wire Wire Line
 	4000 1450 3800 1450
@@
 $EndSheet
 $Comp
-L power:+5V #PWR0105
-U 1 1 614B8AF7
-P 7800 1550
-F 0 "#PWR0105" H 7800 1400 50  0001 C CNN
-F 1 "+5V" H 7815 1723 50  0000 C CNN
-F 2 "" H 7800 1550 50  0001 C CNN
-F 3 "" H 7800 1550 50  0001 C CNN
-	1    7800 1550
-	1    0    0    -1
-$EndComp
-Wire Wire Line
-	7800 1550 7800 1700
-Wire Wire Line
-	7800 1700 8000 1700
-$Comp
 L power:+5V #PWR0106
 U 1 1 614B9875
@@
 Wire Wire Line
 	7850 4050 8050 4050
-NoConn ~ 7800 1900
-Wire Wire Line
-	7800 1900 8000 1900
-Text Label 9200 1900 0    50   ~ 0
-SDA
-Text Label 9200 1700 0    50   ~ 0
-SCL
-Text Label 9200 2100 0    50   ~ 0
-RST
 Text Label 9250 3800 0    50   ~ 0
 SCL
